Commit message: Rebuild CS66 Cell B on teach MDH and swap AG95 for EFG-C65.
Align URDF joint origins/FK-IK with elite_cs66, update tcp_xyz and TCP rotate/maxΔ UI, and expose flange cartesian for viz.

File: src/sensors_arm/static/models/cs66/cs66.urdf (robot description, URDF)
Before this commit: robot CS66urdf, 9 links, 8 joints
Links:
- link gripper_centor_link: geometry collision mesh filename=meshes/EFG-C65.v3.STL; visual mesh filename=meshes/EFG-C65.v3.STL
Joints:
- joint joint1: origin xyz=0 0 0.1625 rpy=0 0 0 -> xyz=0 0 0.162222 rpy=0 0 0
- joint joint2: origin xyz=0 0 0 rpy=1.5708 1.5708 0 -> xyz=0 0 0 rpy=1.5708 0 0
- joint joint3: origin xyz=-0.427 0 0 rpy=0 0 0 -> xyz=-0.427765 0 0 rpy=0 0 0
- joint joint4: origin xyz=-0.3905 0 0.1475 rpy=0 0 -1.5708 -> xyz=-0.391333 0 0.148102 rpy=0 0 0
- joint joint5: origin xyz=0 -0.0965 0 rpy=1.5708 0 0 -> xyz=0 -0.0962059 0 rpy=1.5708 0 0
- joint joint6: origin xyz=0 0.092 0 rpy=-1.5708 0 0 -> xyz=0 0.0948112 0 rpy=-1.5708 0 0
